File: Servos.kicad_sch (KiCad schematic)
At the start: 11 parts, among them SW1 SW_Omron_B3FS, U1 ESP32-S3-DevKitC, U3 PCA9685PW, U4 TCA9545APWR

Commit message: Add most off the stuff
Parts:
- removed C1: 3300u, symbol Device:C_Polarized
- added C10: 100n, symbol Device:C_Small
- added J7: MicroFit3.0_1x2, symbol Connector_Generic:Conn_01x02
- added J9: MoRex_MicroFit-3.0_4x1, symbol Connector_Generic:Conn_01x04
- added R10: 10K, symbol Device:R
- added R11: 10k, symbol Device:R
- added U7: BTT_TMC2209, Project:TMC2209, symbol Project:BTT_TMC2209
- D3: renamed from D1; value SS14 -> 1N5819
- renumbered R4 to R12, R3 to R13, R5 to R7, R2 to R8, R6 to R9, U1 to U5, U3 to U6, U4 to U8
Connections:
- net +3.3V: now also R10.1, U7.15 (VIO)
- net ExtL.SCL: now also U8.9 (SC2); no longer U8.5 (SC0)
- net ExtL.SDA: now also U8.8 (SD2); no longer U8.4 (SD0)
- net ExtL.SIG_MB: now also U6.12 (LED6); no longer U6.6 (LED0)
- net ExtL.SIG_MM: now also U6.13 (LED7); no longer U6.7 (LED1)
- net ExtL.SIG_MS: now also U6.15 (LED8); no longer U6.8 (LED2)
- net ExtR.SCL: now also U8.5 (SC0); no longer U8.9 (SC2)
- net ExtR.SDA: now also U8.4 (SD0); no longer U8.8 (SD2)
- net ExtR.SIG_MB: now also U6.6 (LED0); no longer U6.12 (LED6)
- net ExtR.SIG_MM: now also U6.7 (LED1); no longer U6.13 (LED7)
- net ExtR.SIG_MS: now also U6.8 (LED2); no longer U6.15 (LED8)
- net GND: now also C10.2, J7.2 (Pin_2), R11.2, U7.10 (GND), U7.16 (GND), U7.17 (VREF), U7.2 (MS1), U7.3 (MS2), U7.6 (CLK)
- net IntL.SCL: now also U8.11 (SC3); no longer U8.7 (SC1)
- net IntL.SDA: now also U8.10 (SD3); no longer U8.6 (SD1)
- net IntL.SIG_MB: now also U6.16 (LED9); no longer U6.9 (LED3)
- net IntL.SIG_MM: now also U6.17 (LED10); no longer U6.10 (LED4)
- net IntL.SIG_MS: now also U6.18 (LED11); no longer U6.11 (LED5)
- net IntR.SCL: now also U8.7 (SC1); no longer U8.11 (SC3)
- net IntR.SDA: now also U8.6 (SD1); no longer U8.10 (SD3)
- net IntR.SIG_MB: now also U6.9 (LED3); no longer U6.16 (LED9)
- net IntR.SIG_MM: now also U6.10 (LED4); no longer U6.17 (LED10)
- net IntR.SIG_MS: now also U6.11 (LED5); no longer U6.18 (LED11)
- new net: J9.1 (Pin_1), U7.11 (A2)
- new net: J9.2 (Pin_2), U7.12 (A1)
- new net: J9.3 (Pin_3), U7.13 (B1)
- new net: J9.4 (Pin_4), U7.14 (B2)
- new net +BATT: U7.9 (VM)
- new net Conveyer_DIAG: U7.18 (DIAG)
- new net Conveyer_DIR: U7.8 (DIR)
- new net Conveyer_EN: R11.1, U7.1 (~{EN})
- new net Conveyer_STEP: U7.7 (STEP)
- new net Conveyer_SW: C10.1, J7.1 (Pin_1), R10.2
Other:
- added sheet Grabber Servo (grabber_servo.kicad_sch)
- added sheet Grabber Servo1 (grabber_servo.kicad_sch)
- added sheet Motor_BL (prop.kicad_sch)
- added sheet Motor_BR (prop.kicad_sch)
- added sheet Motor_FL (prop.kicad_sch)
- added sheet Motor_FR (prop.kicad_sch)
- added sheet PumpEL (pump.kicad_sch)
- added sheet PumpER (pump.kicad_sch)
- added sheet PumpIL (pump.kicad_sch)
- added sheet PumpIR (pump.kicad_sch)
- sheet Arm_EL: file arm.kicad_sch -> Arm.kicad_sch
- sheet Arm_ER: file arm.kicad_sch -> Arm.kicad_sch
- sheet Arm_IL: file arm.kicad_sch -> Arm.kicad_sch
- sheet Arm_IR: file arm.kicad_sch -> Arm.kicad_sch
- note added: "Arms"
- note added: "Conveyer stepper"
- note added: "Conveyer switch"
- note added: "Grabber servos"
- note added: "I2C Expander (for coRor captors)"
- note added: "I2C puRRup"
- note added: "Propulsion Motors"
- note added: "Pumps/EV"
- note added: "Servos PWM controRRer"
- note removed: "I2C pullup"
- company: (none) -> Game Team SLSC
- title: (none) -> Logic
- moved on the sheet: R12, R13, R7, R8, R9, SW1, U6, U8

Commit message: Fixes
Parts:
- removed R13: 4.8k, symbol Device:R
- added C18, C23, C24: 100n, symbol Device:C_Small
- added C19: 10u, symbol Device:C_Polarized
- added C21: 470u_LowZ, Capacitor_THT:CP_Radial_D8.0mm_P3.50mm, symbol Device:C_Polarized
- added C22: 10u, symbol Device:C_Small
- added R15: 10k, Resistor_SMD:R_0805_2012Metric_Pad1.20x1.40mm_HandSolder, symbol Device:R
- added R16: 10k, symbol Device:R
- added R19: 1k, symbol Device:R
- added U6: NRF24L01_Breakout, RF_Module:nRF24L01_Breakout, symbol RF:NRF24L01_Breakout
- renumbered C10 to C20, D3 to D5, J7 to J6, J9 to J7, R7 to R11, R8 to R12, R9 to R13, R10 to R14, R12 to R17, R11 to R18, U6 to U7, U7 to U9
Connections:
- net +3.3V: now also C18.1, C19.1, C22.2, C23.2, U6.2 (VCC)
- net +BATT: now also C21.1, C24.2
- net Conveyer_DIR: now also R15.2
- net Conveyer_STEP: now also R16.2
- net GND: now also C18.2, C19.2, C21.2, C22.1, C23.1, C24.1, R15.1, R16.1, U6.1 (GND); no longer U7.23 (~{OE}), U9.17 (VREF)
- net Conveyer_TX: now reaches U9.4 (UART)
- net Conveyer_TX: now also R19.2
- net I2C_Expander_RST: now reaches U8.3 (~{RESET})
- new net Conveyer_RX: R19.1
- new net RF24_CE: U6.3 (CE)
- new net RF24_CSN: U6.4 (~{CSN})
- new net RF24_IRQ: U6.8 (IRQ)
- new net RF24_MISO: U6.7 (MISO)
- new net RF24_MOSI: U6.6 (MOSI)
- new net RF24_SCK: U6.5 (SCK)
- new net Servos_RST: U7.23 (~{OE})
- no-connect marks 46 -> 47
Other:
- note added: "NRF24L01"
- moved on the sheet: J7, R18, U9
