File: alim.kicad_sch (KiCad schematic)
At the start: 8 parts, among them J1 XT60PW-M, J2 XT30PB-M, U2 R-78E5.0-1.0

Commit message: Add most off the stuff
Parts:
- removed D3: P600M, symbol Device:D_Schottky
- removed J1: XT60PW-M, symbol Connector:Conn_01x02_Pin
- removed VR1: XH-M404, symbol Project:Voltage_Regulator_Module
- added C1, C3: 10u, symbol Device:C_Small
- added C2: 22u, Capacitor_SMD:C_0805_2012Metric_Pad1.18x1.45mm_HandSolder, symbol Device:C_Small
- added C4: 47u, symbol Device:C_Small
- added C5, C55, C56, C6, C7: 100n, symbol Device:C_Small
- added C54, C8: 100n, Capacitor_SMD:C_0805_2012Metric_Pad1.18x1.45mm_HandSolder, symbol Device:C_Small
- added D12: 1N4744A, Diode_THT:D_DO-41_SOD81_P10.16mm_Horizontal, symbol Diode:1N47xxA
- added D13: 0805, LED_SMD:LED_0805_2012Metric_Pad1.15x1.40mm_HandSolder, symbol Device:LED
- added J1: Conn_01x02, Connector_AMASS:AMASS_XT60PW-M_1x02_P7.20mm_Horizontal, symbol Connector_Generic:Conn_01x02
- added J3, J4: Conn_01x02, Connector_AMASS:AMASS_XT30UPB-M_1x02_P5.0mm_Vertical, symbol Connector_Generic:Conn_01x02
- added Q9: IRF4905, Package_TO_SOT_THT:TO-220-3_Vertical, symbol Transistor_FET:IRF4905
- added R2: 100R, symbol Device:R_Small
- added R50: 287k, symbol Device:R
- added R51: 60.4k, symbol Device:R
- added R52: 10k, symbol Device:R
- added R53: 100, symbol Device:R
- added U12: TSR3-24120N, Converter_DCDC:Converter_DCDC_TRACO_TSR2-24xxN_TSR2-24xxxN_THT, symbol Regulator_Switching:TSR3-24120N
- added U3: TMCS1100A2QDR, symbol Project:TMCS1100A2QDR
- D2: value LED_Green_3mm -> 0805; footprint (none) -> LED_SMD:LED_0805_2012Metric_Pad1.15x1.40mm_HandSolder; MPN (none) -> APA2106ZGCK; Manufacturer (none) -> Kingbright
- F1: value 15A -> 25A
- J2: symbol Connector:Conn_01x02_Pin -> Connector_Generic:Conn_01x02
- renumbered U2 to U1
Connections:
- net +5V: now also C3.2, C56.2
- net +6V: now also U3.2 (IN-)
- net +BATT: now also J2.2 (Pin_2), C1.2, C2.1, C55.2, C8.1, J3.2 (Pin_2), R50.1, U12.1 (Vin); no longer J2.1 (Pin_1)
- net GND: now also C1.1, C2.2, C3.1, C4.1, C5.1, C54.2, C55.1, C56.1, C6.1, C7.1, C8.2, J1.1 (Pin_1), J3.1 (Pin_1), J4.1 (Pin_1), R51.2, R52.2, R53.2, U12.2 (GND), U3.4 (VREF), U3.6 (GND)
- net at F1.1: now also J1.2 (Pin_2)
- net at F1.2: now also Q9.2 (D); no longer J2.2 (Pin_2)
- new net: D13.1 (K), R53.1
- new net: R2.1, U3.3 (VOUT)
- new net: J4.2 (Pin_2), U3.1 (IN+)
- new net: D12.2 (A), Q9.1 (G), R52.1
- new net: D12.1 (K), J2.1 (Pin_1), Q9.3 (S)
- new net +12V: C4.2, C54.1, U12.3 (Vout)
- new net +3.3V: C6.2, U3.5 (VS)
- new net Batt_Voltage_Led: D13.2 (A)
- new net Batt_Voltage_Sig: C5.2, R50.2, R51.1
- new net ServosCMeasure: C7.2, R2.2
Other:
- note added: "BATT INPUT"
- note added: "Batt watcher"
- note added: "Battery Indicator"
- note added: "Power indicator"
- note added: "Pumps"
- note added: "Rogic ReveR"
- note added: "Servos Power"
- note removed: "INPUT"
- note removed: "Logic level"
- note removed: "Servos level"
- moved on the sheet: D2, F1, R1, U1

Commit message: Fixes
Parts:
- added C10: 2700u_LowZ, Capacitor_THT:CP_Radial_D8.0mm_P3.50mm, symbol Device:C_Polarized
- added C9: 100n, Capacitor_SMD:C_0805_2012Metric_Pad1.18x1.45mm_HandSolder, symbol Device:C_Small
- added D4: 1.5KE8.2A, Diode_THT:D_DO-201AE_P15.24mm_Horizontal, symbol Diode:1.5KExxA
- C11: renamed from C5; footprint (none) -> Capacitor_SMD:C_0805_2012Metric_Pad1.18x1.45mm_HandSolder
- C12: renamed from C6; footprint (none) -> Capacitor_SMD:C_0805_2012Metric_Pad1.18x1.45mm_HandSolder
- C13: renamed from C7; footprint (none) -> Capacitor_SMD:C_0805_2012Metric_Pad1.18x1.45mm_HandSolder
- C2: renamed from C1; footprint (none) -> Capacitor_SMD:C_0805_2012Metric_Pad1.18x1.45mm_HandSolder
- C4: renamed from C55; footprint (none) -> Capacitor_SMD:C_0805_2012Metric_Pad1.18x1.45mm_HandSolder
- C6: renamed from C56; footprint (none) -> Capacitor_SMD:C_0805_2012Metric_Pad1.18x1.45mm_HandSolder
- C7: renamed from C4; footprint (none) -> Capacitor_SMD:C_0805_2012Metric_Pad1.18x1.45mm_HandSolder
- C8: renamed from C3; footprint (none) -> Capacitor_SMD:C_0805_2012Metric_Pad1.18x1.45mm_HandSolder
- D2: value 0805 -> 0805_Green
- D3: renamed from D13; value 0805 -> 0805_Red
- renumbered C2 to C1, C8 to C3, C54 to C5, D12 to D1, J4 to J3, J3 to J4, Q9 to Q1, R52 to R1, R1 to R2, R53 to R3, R50 to R4, R51 to R5, R2 to R6, U12 to U1, U1 to U2
Connections:
- net GND: now also C10.2, C9.1, D4.2 (A2)
- net at J3.2 (Pin_2), U3.1 (IN+): now also C10.1, C9.2, D4.1 (A1)
Other:
- moved on the sheet: C6, C8, J3
