File: arm.kicad_sch (KiCad schematic)
At the start: 7 parts, among them J4 Conn_02x06_Top_Bottom

Commit message: Add most off the stuff
Parts:
- removed C20: 100n, symbol Device:C_Small
- removed C4: 1000u, symbol Device:C_Polarized
- removed J4: Conn_02x06_Top_Bottom, symbol Connector_Generic:Conn_02x07_Top_Bottom
- removed R11, R9: 4.7k, symbol Device:R
- added C11, C14: 100n, Capacitor_SMD:C_0805_2012Metric_Pad1.18x1.45mm_HandSolder, symbol Device:C_Small
- added C13, C17: 470u_LowZ, Capacitor_THT:CP_Radial_D8.0mm_P3.50mm, symbol Device:C_Polarized
- added C15: 470u_LowZ, symbol Device:C_Polarized
- added J10: Molex_MicroFit3.0_02x07, Connector_Molex:Molex_Micro-Fit_3.0_43045-1412_2x07_P3.00mm_Vertical, symbol Connector_Generic:Conn_02x07_Top_Bottom
- added R14, R15: 4.7k, Resistor_SMD:R_0805_2012Metric_Pad1.20x1.40mm_HandSolder, symbol Device:R
- C12, C16: footprint (none) -> Capacitor_SMD:C_0805_2012Metric_Pad1.18x1.45mm_HandSolder
Connections:
- net GNDPWR is gone; now on net GND: C12.2, C16.2
- net +3.3V: now also C11.2, J10.7 (Pin_7), R14.1, R15.2
- net GND: now also C11.1, C13.2, C14.2, C15.2, C17.2, J10.1 (Pin_1), J10.14 (Pin_14), J10.2 (Pin_2), J10.3 (Pin_3)
- net MOT_B: now also J10.4 (Pin_4)
- net MOT_M: now also J10.11 (Pin_11)
- net MOT_S: now also J10.5 (Pin_5)
- net SCL: now also J10.6 (Pin_6), R14.2
- net SDA: now also J10.13 (Pin_13), R15.1
- net V_MOT: now also C13.1, C14.1, C15.1, C17.1, J10.10 (Pin_10), J10.8 (Pin_8), J10.9 (Pin_9)
Other:
- note added: "Torsader - GND / V_MOT (une torsade par servo tous les 3cm) - SCL / GND - SDA / +3.3V Ne pas torsader - MOT_B / MOT_M / MOT_S (ou légèrement autour du GND/V_MOT de son servo)"
- note removed: "Torsader - GNDPWR / V_MOT - MOT_B / MOT_M / MOT_S - SCL / GND - SDA / +3.3V"

Commit message: Fixes
Parts:
- added C25: 10u, Capacitor_SMD:C_0805_2012Metric_Pad1.18x1.45mm_HandSolder, symbol Device:C_Small
- renumbered C11 to C26, C12 to C27, C13 to C28, C14 to C29, C15 to C30, C16 to C31, C17 to C32, J10 to J8, R14 to R20, R15 to R21
Connections:
- net +3.3V: now also C25.2
- net GND: now also C25.1
