File: grabber_servo.kicad_sch (KiCad schematic)
At the start: 3 parts, among them J6 MicroFit3.0_1x3

Commit message: Fixes
Parts:
- renumbered C39 to C73, C41 to C74, J6 to J19
Changed lines of the file:
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@@
 		(dnp no)
 		(fields_autoplaced yes)
-		(property "Reference" "#PWR035"
+		(property "Reference" "#PWR0160"
 			(at 134.62 93.98 0)
 			(effects
@@
 			(project "eurobot-2026-robot-pcb"
 				(path "/b7a41ac4-1d1a-4287-8cea-fdfe5ab5ee00/1a8703d8-5ba0-4c53-bb87-3353758fd726/79cde46c-0510-47ab-a425-44099e6548ad"
-					(reference "#PWR035")
-					(unit 1)
-				)
-				(path "/b7a41ac4-1d1a-4287-8cea-fdfe5ab5ee00/1a8703d8-5ba0-4c53-bb87-3353758fd726/8067320e-3a5b-49b8-9c23-cb84052c5a0d"
-					(reference "#PWR042")
+					(reference "#PWR0160")
+					(unit 1)
+				)
+				(path "/b7a41ac4-1d1a-4287-8cea-fdfe5ab5ee00/1a8703d8-5ba0-4c53-bb87-3353758fd726/8067320e-3a5b-49b8-9c23-cb84052c5a0d"
+					(reference "#PWR0164")
 					(unit 1)
 				)
@@
 		(on_board yes)
 		(dnp no)
-		(property "Reference" "C39"
+		(property "Reference" "C73"
 			(at 130.302 87.376 0)
 			(effects
@@
 			(project "eurobot-2026-robot-pcb"
 				(path "/b7a41ac4-1d1a-4287-8cea-fdfe5ab5ee00/1a8703d8-5ba0-4c53-bb87-3353758fd726/79cde46c-0510-47ab-a425-44099e6548ad"
-					(reference "C39")
-					(unit 1)
-				)
-				(path "/b7a41ac4-1d1a-4287-8cea-fdfe5ab5ee00/1a8703d8-5ba0-4c53-bb87-3353758fd726/8067320e-3a5b-49b8-9c23-cb84052c5a0d"
-					(reference "C43")
+					(reference "C73")
+					(unit 1)
+				)
+				(path "/b7a41ac4-1d1a-4287-8cea-fdfe5ab5ee00/1a8703d8-5ba0-4c53-bb87-3353758fd726/8067320e-3a5b-49b8-9c23-cb84052c5a0d"
+					(reference "C75")
 					(unit 1)
 				)
@@
 		(dnp no)
 		(fields_autoplaced yes)
-		(property "Reference" "#PWR0150"
+		(property "Reference" "#PWR0161"
 			(at 139.7 80.01 0)
 			(effects
@@
 			(project "eurobot-2026-robot-pcb"
 				(path "/b7a41ac4-1d1a-4287-8cea-fdfe5ab5ee00/1a8703d8-5ba0-4c53-bb87-3353758fd726/79cde46c-0510-47ab-a425-44099e6548ad"
-					(reference "#PWR0150")
-					(unit 1)
-				)
-				(path "/b7a41ac4-1d1a-4287-8cea-fdfe5ab5ee00/1a8703d8-5ba0-4c53-bb87-3353758fd726/8067320e-3a5b-49b8-9c23-cb84052c5a0d"
-					(reference "#PWR0152")
+					(reference "#PWR0161")
+					(unit 1)
+				)
+				(path "/b7a41ac4-1d1a-4287-8cea-fdfe5ab5ee00/1a8703d8-5ba0-4c53-bb87-3353758fd726/8067320e-3a5b-49b8-9c23-cb84052c5a0d"
+					(reference "#PWR0165")
 					(unit 1)
 				)
@@
 		(dnp no)
 		(fields_autoplaced yes)
-		(property "Reference" "#PWR0151"
+		(property "Reference" "#PWR0162"
 			(at 146.05 82.55 0)
 			(effects
@@
 			(project "eurobot-2026-robot-pcb"
 				(path "/b7a41ac4-1d1a-4287-8cea-fdfe5ab5ee00/1a8703d8-5ba0-4c53-bb87-3353758fd726/79cde46c-0510-47ab-a425-44099e6548ad"
-					(reference "#PWR0151")
-					(unit 1)
-				)
-				(path "/b7a41ac4-1d1a-4287-8cea-fdfe5ab5ee00/1a8703d8-5ba0-4c53-bb87-3353758fd726/8067320e-3a5b-49b8-9c23-cb84052c5a0d"
-					(reference "#PWR0153")
+					(reference "#PWR0162")
+					(unit 1)
+				)
+				(path "/b7a41ac4-1d1a-4287-8cea-fdfe5ab5ee00/1a8703d8-5ba0-4c53-bb87-3353758fd726/8067320e-3a5b-49b8-9c23-cb84052c5a0d"
+					(reference "#PWR0166")
 					(unit 1)
 				)
@@
 		(dnp no)
 		(fields_autoplaced yes)
-		(property "Reference" "#PWR036"
+		(property "Reference" "#PWR0163"
 			(at 156.21 96.52 0)
 			(effects
@@
 			(project "eurobot-2026-robot-pcb"
 				(path "/b7a41ac4-1d1a-4287-8cea-fdfe5ab5ee00/1a8703d8-5ba0-4c53-bb87-3353758fd726/79cde46c-0510-47ab-a425-44099e6548ad"
-					(reference "#PWR036")
-					(unit 1)
-				)
-				(path "/b7a41ac4-1d1a-4287-8cea-fdfe5ab5ee00/1a8703d8-5ba0-4c53-bb87-3353758fd726/8067320e-3a5b-49b8-9c23-cb84052c5a0d"
-					(reference "#PWR043")
+					(reference "#PWR0163")
+					(unit 1)
+				)
+				(path "/b7a41ac4-1d1a-4287-8cea-fdfe5ab5ee00/1a8703d8-5ba0-4c53-bb87-3353758fd726/8067320e-3a5b-49b8-9c23-cb84052c5a0d"
+					(reference "#PWR0167")
 					(unit 1)
 				)
@@
 		(dnp no)
 		(fields_autoplaced yes)
-		(property "Reference" "J6"
+		(property "Reference" "J19"
 			(at 170.18 92.7099 0)
 			(effects
@@
 			(project "eurobot-2026-robot-pcb"
 				(path "/b7a41ac4-1d1a-4287-8cea-fdfe5ab5ee00/1a8703d8-5ba0-4c53-bb87-3353758fd726/79cde46c-0510-47ab-a425-44099e6548ad"
-					(reference "J6")
-					(unit 1)
-				)
-				(path "/b7a41ac4-1d1a-4287-8cea-fdfe5ab5ee00/1a8703d8-5ba0-4c53-bb87-3353758fd726/8067320e-3a5b-49b8-9c23-cb84052c5a0d"
-					(reference "J8")
+					(reference "J19")
+					(unit 1)
+				)
+				(path "/b7a41ac4-1d1a-4287-8cea-fdfe5ab5ee00/1a8703d8-5ba0-4c53-bb87-3353758fd726/8067320e-3a5b-49b8-9c23-cb84052c5a0d"
+					(reference "J20")
 					(unit 1)
 				)
@@
 		(dnp no)
 		(fields_autoplaced yes)
-		(property "Reference" "C41"
+		(property "Reference" "C74"
 			(at 148.59 90.1635 0)
 			(effects
@@
 			(project "eurobot-2026-robot-pcb"
 				(path "/b7a41ac4-1d1a-4287-8cea-fdfe5ab5ee00/1a8703d8-5ba0-4c53-bb87-3353758fd726/79cde46c-0510-47ab-a425-44099e6548ad"
-					(reference "C41")
-					(unit 1)
-				)
-				(path "/b7a41ac4-1d1a-4287-8cea-fdfe5ab5ee00/1a8703d8-5ba0-4c53-bb87-3353758fd726/8067320e-3a5b-49b8-9c23-cb84052c5a0d"
-					(reference "C53")
-					(unit 1)
-				)
+					(reference "C74")
+					(unit 1)
+				)
+				(path "/b7a41ac4-1d1a-4287-8cea-fdfe5ab5ee00/1a8703d8-5ba0-4c53-bb87-3353758fd726/8067320e-3a5b-49b8-9c23-cb84052c5a0d"
+					(reference "C76")
+					(unit 1)
+				)
