File: prop.kicad_sch (KiCad schematic)
At the start: 8 parts, among them J5 MoRex_MicroFit-3.0_4x1, U4 BTT_TMC5160T_Pro

Commit message: Fixes
Parts:
- added C15: 10u, symbol Device:C_Small
- added C17: 100n, Capacitor_SMD:C_0805_2012Metric_Pad1.18x1.45mm_HandSolder, symbol Device:C_Small
- renumbered C49 to C14, C9 to C16, R6 to R10, R3 to R7, R4 to R8, R5 to R9
Connections:
- net +3.3V: now also C17.1
- net +BATT: now also C15.2
- net GND: now also C15.1, C17.2
Other:
- moved on the sheet: C14, C16
