File: pump.kicad_sch (KiCad schematic)
At the start: 10 parts, among them J17 MicroFit3.0_2x2, Q1 IRRZ44N, Q2 IRRZ44N

Commit message: Fixes
Parts:
- renumbered C45 to C69, D4 to D6, D5 to D7, J17 to J15, Q1 to Q2, Q2 to Q3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
