File: sheets/arm.kicad_sch (KiCad schematic)
At the start: 11 parts, among them J8 Molex_MicroFit3.0_02x07

Commit message: Add CB1-P-12V relay footprint, 3D model, and symbols
Added CB1-P-12V.stp 3D model and CB1P12V.kicad_mod footprint to the libs directory. Updated libs/sym.kicad_sym and multiple schematic sheets to include and reference the new relay. Adjusted eurobot-2026-robot-pcb.kicad_pro BOM and group settings to support new components.
Parts:
- renumbered C28 to C29, C32 to C31, C27 to C32, C29 to C33, C31 to C34, C26 to C35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
