File: sheets/grabber_servo.kicad_sch (KiCad schematic)
At the start: 3 parts, among them J19 MicroFit3.0_1x3

Commit message: Add CB1-P-12V relay footprint, 3D model, and symbols
Added CB1-P-12V.stp 3D model and CB1P12V.kicad_mod footprint to the libs directory. Updated libs/sym.kicad_sym and multiple schematic sheets to include and reference the new relay. Adjusted eurobot-2026-robot-pcb.kicad_pro BOM and group settings to support new components.
Parts:
- renumbered C73 to C81, C74 to C82
Changed lines of the file:
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@@
 		(dnp no)
 		(fields_autoplaced yes)
-		(property "Reference" "#PWR0160"
+		(property "Reference" "#PWR0173"
 			(at 134.62 93.98 0)
 			(effects
@@
 			(project "eurobot-2026-robot-pcb"
 				(path "/b7a41ac4-1d1a-4287-8cea-fdfe5ab5ee00/1a8703d8-5ba0-4c53-bb87-3353758fd726/79cde46c-0510-47ab-a425-44099e6548ad"
-					(reference "#PWR0160")
-					(unit 1)
-				)
-				(path "/b7a41ac4-1d1a-4287-8cea-fdfe5ab5ee00/1a8703d8-5ba0-4c53-bb87-3353758fd726/8067320e-3a5b-49b8-9c23-cb84052c5a0d"
-					(reference "#PWR0164")
+					(reference "#PWR0173")
+					(unit 1)
+				)
+				(path "/b7a41ac4-1d1a-4287-8cea-fdfe5ab5ee00/1a8703d8-5ba0-4c53-bb87-3353758fd726/8067320e-3a5b-49b8-9c23-cb84052c5a0d"
+					(reference "#PWR0177")
 					(unit 1)
 				)
@@
 		(on_board yes)
 		(dnp no)
-		(property "Reference" "C73"
+		(property "Reference" "C81"
 			(at 130.302 87.376 0)
 			(effects
@@
 			(project "eurobot-2026-robot-pcb"
 				(path "/b7a41ac4-1d1a-4287-8cea-fdfe5ab5ee00/1a8703d8-5ba0-4c53-bb87-3353758fd726/79cde46c-0510-47ab-a425-44099e6548ad"
-					(reference "C73")
-					(unit 1)
-				)
-				(path "/b7a41ac4-1d1a-4287-8cea-fdfe5ab5ee00/1a8703d8-5ba0-4c53-bb87-3353758fd726/8067320e-3a5b-49b8-9c23-cb84052c5a0d"
-					(reference "C75")
+					(reference "C81")
+					(unit 1)
+				)
+				(path "/b7a41ac4-1d1a-4287-8cea-fdfe5ab5ee00/1a8703d8-5ba0-4c53-bb87-3353758fd726/8067320e-3a5b-49b8-9c23-cb84052c5a0d"
+					(reference "C83")
 					(unit 1)
 				)
@@
 		(dnp no)
 		(fields_autoplaced yes)
-		(property "Reference" "#PWR0161"
+		(property "Reference" "#PWR0171"
 			(at 139.7 80.01 0)
 			(effects
@@
 			(project "eurobot-2026-robot-pcb"
 				(path "/b7a41ac4-1d1a-4287-8cea-fdfe5ab5ee00/1a8703d8-5ba0-4c53-bb87-3353758fd726/79cde46c-0510-47ab-a425-44099e6548ad"
-					(reference "#PWR0161")
-					(unit 1)
-				)
-				(path "/b7a41ac4-1d1a-4287-8cea-fdfe5ab5ee00/1a8703d8-5ba0-4c53-bb87-3353758fd726/8067320e-3a5b-49b8-9c23-cb84052c5a0d"
-					(reference "#PWR0165")
+					(reference "#PWR0171")
+					(unit 1)
+				)
+				(path "/b7a41ac4-1d1a-4287-8cea-fdfe5ab5ee00/1a8703d8-5ba0-4c53-bb87-3353758fd726/8067320e-3a5b-49b8-9c23-cb84052c5a0d"
+					(reference "#PWR0175")
 					(unit 1)
 				)
@@
 		(dnp no)
 		(fields_autoplaced yes)
-		(property "Reference" "#PWR0162"
+		(property "Reference" "#PWR0172"
 			(at 146.05 82.55 0)
 			(effects
@@
 			(project "eurobot-2026-robot-pcb"
 				(path "/b7a41ac4-1d1a-4287-8cea-fdfe5ab5ee00/1a8703d8-5ba0-4c53-bb87-3353758fd726/79cde46c-0510-47ab-a425-44099e6548ad"
-					(reference "#PWR0162")
-					(unit 1)
-				)
-				(path "/b7a41ac4-1d1a-4287-8cea-fdfe5ab5ee00/1a8703d8-5ba0-4c53-bb87-3353758fd726/8067320e-3a5b-49b8-9c23-cb84052c5a0d"
-					(reference "#PWR0166")
+					(reference "#PWR0172")
+					(unit 1)
+				)
+				(path "/b7a41ac4-1d1a-4287-8cea-fdfe5ab5ee00/1a8703d8-5ba0-4c53-bb87-3353758fd726/8067320e-3a5b-49b8-9c23-cb84052c5a0d"
+					(reference "#PWR0176")
 					(unit 1)
 				)
@@
 		(dnp no)
 		(fields_autoplaced yes)
-		(property "Reference" "#PWR0163"
+		(property "Reference" "#PWR0174"
 			(at 156.21 96.52 0)
 			(effects
@@
 			(project "eurobot-2026-robot-pcb"
 				(path "/b7a41ac4-1d1a-4287-8cea-fdfe5ab5ee00/1a8703d8-5ba0-4c53-bb87-3353758fd726/79cde46c-0510-47ab-a425-44099e6548ad"
-					(reference "#PWR0163")
-					(unit 1)
-				)
-				(path "/b7a41ac4-1d1a-4287-8cea-fdfe5ab5ee00/1a8703d8-5ba0-4c53-bb87-3353758fd726/8067320e-3a5b-49b8-9c23-cb84052c5a0d"
-					(reference "#PWR0167")
+					(reference "#PWR0174")
+					(unit 1)
+				)
+				(path "/b7a41ac4-1d1a-4287-8cea-fdfe5ab5ee00/1a8703d8-5ba0-4c53-bb87-3353758fd726/8067320e-3a5b-49b8-9c23-cb84052c5a0d"
+					(reference "#PWR0178")
 					(unit 1)
 				)
@@
 		(dnp no)
 		(fields_autoplaced yes)
-		(property "Reference" "C74"
+		(property "Reference" "C82"
 			(at 148.59 90.1635 0)
 			(effects
@@
 			(project "eurobot-2026-robot-pcb"
 				(path "/b7a41ac4-1d1a-4287-8cea-fdfe5ab5ee00/1a8703d8-5ba0-4c53-bb87-3353758fd726/79cde46c-0510-47ab-a425-44099e6548ad"
-					(reference "C74")
-					(unit 1)
-				)
-				(path "/b7a41ac4-1d1a-4287-8cea-fdfe5ab5ee00/1a8703d8-5ba0-4c53-bb87-3353758fd726/8067320e-3a5b-49b8-9c23-cb84052c5a0d"
-					(reference "C76")
-					(unit 1)
-				)
+					(reference "C82")
+					(unit 1)
+				)
+				(path "/b7a41ac4-1d1a-4287-8cea-fdfe5ab5ee00/1a8703d8-5ba0-4c53-bb87-3353758fd726/8067320e-3a5b-49b8-9c23-cb84052c5a0d"
+					(reference "C84")
+					(unit 1)
+				)
