File: sheets/prop.kicad_sch (KiCad schematic)
At the start: 10 parts, among them J5 MoRex_MicroFit-3.0_4x1, U4 BTT_TMC5160T_Pro

Commit message: Add CB1-P-12V relay footprint, 3D model, and symbols
Added CB1-P-12V.stp 3D model and CB1P12V.kicad_mod footprint to the libs directory. Updated libs/sym.kicad_sym and multiple schematic sheets to include and reference the new relay. Adjusted eurobot-2026-robot-pcb.kicad_pro BOM and group settings to support new components.
Parts:
- C18: renamed from C14; MPN EEU-FR1E471L -> EEUFR1C182L
- renumbered C17 to C19, C15 to C20, C16 to C21, R8 to R11, R9 to R12, R7 to R13, R10 to R14, U4 to U6
