File: sheets/pump.kicad_sch (KiCad schematic)
At the start: 10 parts, among them J15 MicroFit3.0_2x2, Q2 IRRZ44N, Q3 IRRZ44N

Commit message: Add relay for BAU + fixes
Parts:
- Q2, Q3: value IRRZ44N -> IRLZ44N
Changed lines of the file:
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@@
 			)
 		)
-		(property "Value" "IRRZ44N"
+		(property "Value" "IRLZ44N"
 			(at 81.28 52.07 90)
 			(effects
@@
 			)
 		)
-		(property "Value" "IRRZ44N"
+		(property "Value" "IRLZ44N"
 			(at 125.73 53.34 90)
 			(effects

Commit message: Add CB1-P-12V relay footprint, 3D model, and symbols
Added CB1-P-12V.stp 3D model and CB1P12V.kicad_mod footprint to the libs directory. Updated libs/sym.kicad_sym and multiple schematic sheets to include and reference the new relay. Adjusted eurobot-2026-robot-pcb.kicad_pro BOM and group settings to support new components.
Parts:
- added C74: 100n, symbol Device:C
- C73: renamed from C69; value 470u_LowZ -> 47u_LowZ; footprint Capacitor_THT:CP_Radial_D8.0mm_P3.50mm -> Capacitor_THT:CP_Radial_D5.0mm_P2.00mm; MPN EEU-FR1E471L -> EEUFR1E470
- D8: renamed from D6; value 1N5819 -> SS24
- D9: renamed from D7; value 1N5819 -> SS24
- renumbered Q2 to Q3, Q3 to Q4, R41 to R44, R43 to R45, R40 to R46, R42 to R47
Connections:
- net GND: now also C74.1
- net +12V renamed Vin
- net Vin: now also C74.2
Other:
- moved on the sheet: C73
